File: PCB_v2_KiCAD/HarveyBehaviorPCB_v2.kicad_sch (KiCad schematic)
At the start: 67 parts, among them IC1 LT1490A, IC3 40106N, J1 POWER_JACKPTH, J10 M01SMTSO-256-ET-0.165DIA, J11 M01SMTSO-256-ET-0.165DIA, J12 Conn_01x07, J13 Conn_01x07, J14 I2C_STANDARDQWIIC, J15 Valve 1, J16 Valve 1 Switch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

Commit message: Update BOM for v2.0
Parts:
- C1: symbol HarveyBehaviorPCB_v2-eagle-import:CAP_POLPTH2 -> Device:C_Polarized_US
- C2: value C_Polarized_US -> 100nF
Changed lines of the file:
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@@
 	(wire
 		(pts
-			(xy 354.33 35.56) (xy 356.87 35.56)
+			(xy 354.33 43.18) (xy 356.87 43.18)
 		)
 		(stroke
@@
 	(wire
 		(pts
-			(xy 354.33 43.18) (xy 354.33 35.56)
-		)
-		(stroke
-			(width 0)
-			(type default)
-		)
-	)
-	(wire
-		(pts
 			(xy 195.58 162.56) (xy 198.12 162.56)
 		)
@@
 	)
 	(label "LICK_1"
-		(at 356.87 35.56 0)
+		(at 356.87 43.18 0)
 		(fields_autoplaced yes)
 		(effects
@@
 			)
 		)
-		(property "Value" "C_Polarized_US"
+		(property "Value" "100nF"
 			(at 325.755 102.87 0)
 			(effects
@@
 				)
 				(justify left)
-				(hide yes)
 			)
 		)
@@
 	)
 	(symbol
-		(lib_id "HarveyBehaviorPCB_v2-eagle-import:CAP_POLPTH2")
-		(at 325.12 48.26 0)
+		(lib_id "Device:C_Polarized_US")
+		(at 325.12 49.53 0)
 		(unit 1)
 		(exclude_from_sim no)
@@
 		(dnp no)
 		(property "Reference" "C1"
-			(at 326.136 47.625 0)
+			(at 326.136 48.006 0)
 			(effects
 				(font
-					(size 1.778 1.5113)
+					(size 1.27 1.27)
 				)
 				(justify left bottom)
@@
 		)
 		(property "Value" "100nF"
-			(at 326.136 52.451 0)
+			(at 326.136 53.721 0)
 			(effects
 				(font
-					(size 1.778 1.5113)
+					(size 1.27 1.27)
 				)
 				(justify left bottom)
@@
 		)
 		(property "Footprint" "HarveyBehaviorPCB_v2:CPOL-RADIAL-10UF-25V"
-			(at 325.12 48.26 0)
+			(at 325.12 49.53 0)
 			(effects
 				(font
@@
 			)
 		)
-		(property "Datasheet" ""
-			(at 325.12 48.26 0)
+		(property "Datasheet" "~"
+			(at 325.12 49.53 0)
 			(effects
 				(font
@@
 			)
 		)
-		(property "Description" ""
-			(at 325.12 48.26 0)
+		(property "Description" "Polarized capacitor, US symbol"
+			(at 325.12 49.53 0)
 			(effects
 				(font
