File: PCB_v2_KiCAD/HarveyBehaviorPCB_v2.kicad_pcb (KiCad board)
At the start: 2 copper layers, 203.2 x 125.7 mm, 68 parts, among them IC1 LT1490A, IC3 40106N, J1 POWER_JACKPTH, J10 M01SMTSO-256-ET-0.165DIA, J11 M01SMTSO-256-ET-0.165DIA, J12 Conn_01x07, J13 Conn_01x07, J14 I2C_STANDARDQWIIC, J15 Valve 1, J16 Valve 1 Switch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

Commit message: Make Gerbers for v2.0
Other:
- board text added: "LP filters for Vel-Y/R/P"
- board text added: "Lick and photodiode circuits"
- board text added: "User 3/4 voltage-limiting circuit"
- board text removed: "LP Filters for Vel Y/R/P"
- board text removed: "Lick and Photodiode circuits"
- board text removed: "User 3/4 Voltage-limiting circuit"
Changed lines of the file:
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@@
 		)
 	)
-	(gr_text "Lick and Photodiode circuits"
+	(gr_text "Lick and photodiode circuits"
 		(at 140.716 68.326 0)
 		(layer "F.SilkS")
@@
 		)
 	)
-	(gr_text "User 3/4 Voltage-limiting circuit"
+	(gr_text "User 3/4 voltage-limiting circuit"
 		(at 48.26 62.738 0)
 		(layer "F.SilkS")
@@
 		)
 	)
-	(gr_text "LP Filters for Vel Y/R/P"
+	(gr_text "LP filters for Vel-Y/R/P"
 		(at 83.566 129.286 90)
 		(layer "F.SilkS")

Commit message: [PCB] Increase width of copper pads on a few footprints; v2.0 -> v2.01
Other:
- board text added: "Harvey Lab Behavior Circuit v2.01 • OM • Dec 2024"
- board text removed: "Harvey Lab Behavior Circuit v2.0 • OM • Sept 2024"
Changed lines of the file:
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@@
 			(layer "F.Fab")
 		)
+		(fp_text user "MAXIMUM_PACKAGE_HEIGHT:_17.5_MM"
+			(at -17.44998 11.840002 -90)
+			(unlocked yes)
+			(layer "Cmts.User")
+			(effects
+				(font
+					(size 1 1)
+					(thickness 0.15)
+				)
+			)
+		)
+		(fp_text user "NOTE"
+			(at -17.44998 9.300002 -90)
+			(unlocked yes)
+			(layer "Cmts.User")
+			(effects
+				(font
+					(size 1 1)
+					(thickness 0.15)
+				)
+			)
+		)
+		(fp_text user "MATTE_TIN_PLATING,_TRAY_PACKAGING"
+			(at -7.499999 -12.699998 -90)
+			(unlocked yes)
+			(layer "F.Fab")
+			(effects
+				(font
+					(size 1 1)
+					(thickness 0.15)
+				)
+			)
+		)
+		(fp_text user "MINI_LOCK_W/B_SR_VERT_PLUG_ASSY_-7_CKT"
+			(at -7.499999 -15.239997 -90)
+			(unlocked yes)
+			(layer "F.Fab")
+			(effects
+				(font
+					(size 1 1)
+					(thickness 0.15)
+				)
+			)
+		)
+		(fp_text user "${REFERENCE}"
+			(at -7.499998 -8.89 -90)
+			(unlocked yes)
+			(layer "F.Fab")
+			(effects
+				(font
+					(size 1 1)
+					(thickness 0.15)
+				)
+			)
+		)
+		(fp_text user "535170730"
+			(at -7.499999 -17.779997 -90)
+			(unlocked yes)
+			(layer "F.Fab")
+			(effects
+				(font
+					(size 1 1)
+					(thickness 0.15)
+				)
+			)
+		)
 		(pad "" np_thru_hole circle
 			(at 1.6 2.2 270)
 			(size 1.2 1.2)
 			(drill 1.2)
-			(layers "*.Mask")
+			(layers "F&B.Cu" "*.Mask")
 		)
 		(pad "1" thru_hole rect
 			(at 0 0 270)
-			(size 1.05 1.05)
+			(size 1.524 1.524)
 			(drill 0.7)
 			(layers "*.Cu" "*.Mask")
@@
 		(pad "2" thru_hole circle
 			(at -2.5 0 270)
-			(size 1.05 1.05)
+			(size 1.524 1.524)
 			(drill 0.7)
 			(layers "*.Cu" "*.Mask")
@@
 		(pad "3" thru_hole circle
 			(at -5 0 270)
-			(size 1.05 1.05)
+			(size 1.524 1.524)
 			(drill 0.7)
 			(layers "*.Cu" "*.Mask")
@@
 		(pad "4" thru_hole circle
 			(at -7.5 0 270)
-			(size 1.05 1.05)
+			(size 1.524 1.524)
 			(drill 0.7)
 			(layers "*.Cu" "*.Mask")
@@
 		(pad "5" thru_hole circle
 			(at -10 0 270)
-			(size 1.05 1.05)
+			(size 1.524 1.524)
 			(drill 0.7)
 			(layers "*.Cu" "*.Mask")
@@
 		(pad "6" thru_hole circle
 			(at -12.5 0 270)
-			(size 1.05 1.05)
+			(size 1.524 1.524)
 			(drill 0.7)
 			(layers "*.Cu" "*.Mask")
@@
 		(pad "7" thru_hole circle
 			(at -15 0 270)
-			(size 1.05 1.05)
+			(size 1.524 1.524)
 			(drill 0.7)
 			(layers "*.Cu" "*.Mask")
@@
 			(layer "F.Fab")
 		)
+		(fp_text user "MAXIMUM_PACKAGE_HEIGHT:_17.5_MM"
+			(at -17.44998 11.840002 -90)
+			(unlocked yes)
+			(layer "Cmts.User")
+			(effects
+				(font
+					(size 1 1)
+					(thickness 0.15)
+				)
+			)
+		)
+		(fp_text user "NOTE"
+			(at -17.44998 9.300002 -90)
+			(unlocked yes)
+			(layer "Cmts.User")
+			(effects
+				(font
+					(size 1 1)
+					(thickness 0.15)
+				)
+			)
+		)
+		(fp_text user "MINI_LOCK_W/B_SR_VERT_PLUG_ASSY_-7_CKT"
+			(at -7.499999 -15.239997 -90)
+			(unlocked yes)
+			(layer "F.Fab")
+			(effects
+				(font
+					(size 1 1)
+					(thickness 0.15)
+				)
+			)
+		)
+		(fp_text user "${REFERENCE}"
+			(at -7.499998 -8.89 -90)
+			(unlocked yes)
+			(layer "F.Fab")
+			(effects
+				(font
+					(size 1 1)
+					(thickness 0.15)
+				)
+			)
+		)
+		(fp_text user "535170730"
+			(at -7.499999 -17.779997 -90)
+			(unlocked yes)
+			(layer "F.Fab")
+			(effects
+				(font
+					(size 1 1)
+					(thickness 0.15)
+				)
+			)
+		)
+		(fp_text user "MATTE_TIN_PLATING,_TRAY_PACKAGING"
+			(at -7.499999 -12.699998 -90)
+			(unlocked yes)
+			(layer "F.Fab")
+			(effects
+				(font
+					(size 1 1)
+					(thickness 0.15)
+				)
+			)
+		)
 		(pad "" np_thru_hole circle
 			(at 1.6 2.2 270)
@@
 		(pad "1" thru_hole rect
 			(at 0 0 270)
-			(size 1.05 1.05)
+			(size 1.524 1.524)
 			(drill 0.7)
 			(layers "*.Cu" "*.Mask")
@@
 		(pad "2" thru_hole circle
 			(at -2.5 0 270)
-			(size 1.05 1.05)
+			(size 1.524 1.524)
 			(drill 0.7)
 			(layers "*.Cu" "*.Mask")
@@
 		(pad "3" thru_hole circle
 			(at -5 0 270)
-			(size 1.05 1.05)
+			(size 1.524 1.524)
 			(drill 0.7)
 			(layers "*.Cu" "*.Mask")
@@
 		(pad "4" thru_hole circle
 			(at -7.5 0 270)
-			(size 1.05 1.05)
+			(size 1.524 1.524)
 			(drill 0.7)
 			(layers "*.Cu" "*.Mask")
@@
 		(pad "5" thru_hole circle
 			(at -10 0 270)
-			(size 1.05 1.05)
+			(size 1.524 1.524)
 			(drill 0.7)
 			(layers "*.Cu" "*.Mask")
@@
 		(pad "6" thru_hole circle
 			(at -12.5 0 270)
-			(size 1.05 1.05)
+			(size 1.524 1.524)
 			(drill 0.7)
 			(layers "*.Cu" "*.Mask")
@@
 		(pad "7" thru_hole circle
 			(at -15 0 270)
-			(size 1.05 1.05)
+			(size 1.524 1.524)
 			(drill 0.7)
 			(layers "*.Cu" "*.Mask")
@@
 		(pad "0" thru_hole circle
 			(at -7.62 -13.97 180)
-			(size 1.4478 1.4478)
+			(size 1.651 1.651)
 			(drill 0.9652)
 			(layers "*.Cu" "*.Mask")
@@
 		(pad "1" thru_hole circle
 			(at -7.62 -11.43 180)
-			(size 1.4478 1.4478)
+			(size 1.651 1.651)
 			(drill 0.9652)
 			(layers "*.Cu" "*.Mask")
@@
 		(pad "2" thru_hole circle
 			(at -7.62 -8.89 180)
-			(size 1.4478 1.4478)
+			(size 1.651 1.651)
 			(drill 0.9652)
 			(layers "*.Cu" "*.Mask")
@@
 		(pad "3" thru_hole circle
 			(at -7.62 -6.35 180)
-			(size 1.4478 1.4478)
+			(size 1.651 1.651)
 			(drill 0.9652)
 			(layers "*.Cu" "*.Mask")
@@
 		(pad "3.3V" thru_hole circle
 			(at 7.62 -11.43 180)
-			(size 1.4478 1.4478)
+			(size 1.651 1.651)
 			(drill 0.9652)
 			(layers "*.Cu" "*.Mask")
@@
 		(pad "4" thru_hole circle
 			(at -7.62 -3.81 180)
-			(size 1.4478 1.4478)
+			(size 1.651 1.651)
 			(drill 0.9652)
 			(layers "*.Cu" "*.Mask")
@@
 		(pad "5" thru_hole circle
 			(at -7.62 -1.27 180)
-			(size 1.4478 1.4478)
+			(size 1.651 1.651)
 			(drill 0.9652)
 			(layers "*.Cu" "*.Mask")
@@
 		(pad "6" thru_hole circle
 			(at -7.62 1.27 180)
-			(size 1.4478 1.4478)
+			(size 1.651 1.651)
 			(drill 0.9652)
 			(layers "*.Cu" "*.Mask")
@@
 		(pad "7" thru_hole circle
 			(at -7.62 3.81 180)
-			(size 1.4478 1.4478)
+			(size 1.651 1.651)
 			(drill 0.9652)
 			(layers "*.Cu" "*.Mask")
@@
 		(pad "8" thru_hole circle
 			(at -7.62 6.35 180)
-			(size 1.4478 1.4478)
+			(size 1.651 1.651)
 			(drill 0.9652)
 			(layers "*.Cu" "*.Mask")
@@
 		(pad "9" thru_hole circle
 			(at -7.62 8.89 180)
-			(size 1.4478 1.4478)
+			(size 1.651 1.651)
 			(drill 0.9652)
 			(layers "*.Cu" "*.Mask")
@@
 		(pad "10" thru_hole circle
 			(at -7.62 11.43 180)
-			(size 1.4478 1.4478)
+			(size 1.651 1.651)
 			(drill 0.9652)
 			(layers "*.Cu" "*.Mask")
@@
 		(pad "11" thru_hole circle
 			(at -7.62 13.97 180)
-			(size 1.4478 1.4478)
+			(size 1.651 1.651)
 			(drill 0.9652)
 			(layers "*.Cu" "*.Mask")
@@
 		(pad "12" thru_hole circle
 			(at -7.62 16.51 180)
-			(size 1.4478 1.4478)
+			(size 1.651 1.651)
 			(drill 0.9652)
 			(layers "*.Cu" "*.Mask")
@@
 		(pad "13" thru_hole circle
 			(at 7.62 16.51 180)
-			(size 1.4478 1.4478)
+			(size 1.651 1.651)
 			(drill 0.9652)
 			(layers "*.Cu" "*.Mask")
@@
 		(pad "14/A0" thru_hole circle
 			(at 7.62 13.97 180)
-			(size 1.4478 1.4478)
+			(size 1.651 1.651)
 			(drill 0.9652)
 			(layers "*.Cu" "*.Mask")
@@
 		(pad "15/A1" thru_hole circle
 			(at 7.62 11.43 180)
-			(size 1.4478 1.4478)
+			(size 1.651 1.651)
 			(drill 0.9652)
 			(layers "*.Cu" "*.Mask")
@@
 		(pad "16/A2" thru_hole circle
 			(at 7.62 8.89 180)
-			(size 1.4478 1.4478)
+			(size 1.651 1.651)
 			(drill 0.9652)
 			(layers "*.Cu" "*.Mask")
@@
 		(pad "17/A3" thru_hole circle
 			(at 7.62 6.35 180)
-			(size 1.4478 1.4478)
+			(size 1.651 1.651)
 			(drill 0.9652)
 			(layers "*.Cu" "*.Mask")
@@
 		(pad "18/A4" thru_hole circle
 			(at 7.62 3.81 180)
-			(size 1.4478 1.4478)
+			(size 1.651 1.651)
 			(drill 0.9652)
 			(layers "*.Cu" "*.Mask")
@@
 		(pad "19/A5" thru_hole circle
 			(at 7.62 1.27 180)
-			(size 1.4478 1.4478)
+			(size 1.651 1.651)
 			(drill 0.9652)
 			(layers "*.Cu" "*.Mask")
@@
 		(pad "20/A6" thru_hole circle
 			(at 7.62 -1.27 180)
-			(size 1.4478 1.4478)
+			(size 1.651 1.651)
 			(drill 0.9652)
 			(layers "*.Cu" "*.Mask")
@@
 		(pad "21/A7" thru_hole circle
 			(at 7.62 -3.81 180)
-			(size 1.4478 1.4478)
+			(size 1.651 1.651)
 			(drill 0.9652)
 			(layers "*.Cu" "*.Mask")
@@
 		(pad "22/A8" thru_hole circle
 			(at 7.62 -6.35 180)
-			(size 1.4478 1.4478)
+			(size 1.651 1.651)
 			(drill 0.9652)
 			(layers "*.Cu" "*.Mask")
@@
 		(pad "23/A9" thru_hole circle
 			(at 7.62 -8.89 180)
-			(size 1.4478 1.4478)
+			(size 1.651 1.651)
 			(drill 0.9652)
 			(layers "*.Cu" "*.Mask")
@@
 		(pad "AGND" thru_hole circle
 			(at 7.62 -13.97 180)
-			(size 1.4478 1.4478)
+			(size 1.651 1.651)
 			(drill 0.9652)
 			(layers "*.Cu" "*.Mask")
@@
 		(pad "GND" thru_hole circle
 			(at -7.62 -16.51 180)
-			(size 1.4478 1.4478)
+			(size 1.651 1.651)
 			(drill 0.9652)
 			(layers "*.Cu" "*.Mask")
@@
 		(pad "VIN" thru_hole circle
 			(at 7.62 -16.51 180)
-			(size 1.4478 1.4478)
+			(size 1.651 1.651)
 			(drill 0.9652)
 			(layers "*.Cu" "*.Mask")
@@
 		)
 	)
-	(gr_text "Harvey Lab Behavior Circuit\nv2.0  •  OM  •  Sept 2024"
+	(gr_text "Harvey Lab Behavior Circuit\nv2.01  •  OM  •  Dec 2024"
 		(at 151.5999 124.7394 0)
 		(layer "F.SilkS")
